Commit message: fix(sim): correct gripper normalization and replace nonexistent Isaac Lab mdp terms
Verified every uncertain Isaac Lab API against the v2.3.2 source (tag 37ddf62,
shallow clone, no Isaac Sim install needed) and fixed what was actually broken.

Unit conversion (the one silent-failure path):
- The gripper used its mechanical range (100deg -> 100%) instead of lerobot's
  encoder-tick normalization. OmxFollower.calibrate() writes range_min=0 and
  range_max=4095 for every motor including the gripper, so RANGE_0_100 spans one
  full revolution: 100deg -> 27.8%, i.e. pct = q * 50/pi, exactly half the arm
  coefficient. Only the zero reference still needs hardware confirmation.
- Test expectations no longer derive from JOINT_LIMITS_RAD. Sharing that premise
  between implementation and test is what let the wrong formula pass in the first
  place, so the boundary values are now hardcoded from the tick math.

Nonexistent mdp references (would AttributeError at manager init):
- object_is_grasped, object_lift_height and root_pose_w do not exist in v2.3.2.
- object_ee_distance lives only in the lift task and reads a single
  FrameTransformer target, so it cannot express bimanual semantics no matter how
  many body names it is handed.
- Added lelab_sim/envs/mdp/ with three bimanual-explicit terms. The reach reward
  multiplies per-arm tanh kernels so a one-arm solution cannot score, and the
  grasp reward shares both_grippers_touching with collect_rollouts so the training
  signal and the episode-acceptance criterion cannot drift apart.
- Split root_pose_w into root_pos_w plus root_quat_w. Observation is now 60-dim
  as the design specifies.

Also restored the reset-mode joint reset event, rewrote package:// mesh URIs to
paths relative to the generated URDF, derived mimic joint limits from their target
joint, and stopped treating a step-cap hit as an episode end since the env is not
reset there and the trajectory would be a fragment.

Confirmed the rest of the API surface was already correct: body_pose_w returns
7*num_bodies, decimation belongs to ManagerBasedEnvCfg not SimulationCfg,
configclass injects __post_init__ so re-calling it is safe, force_matrix_w really
can be None, and RelativeJointPositionActionCfg has use_zero_offset rather than
use_default_offset.

Verified: 4 sim tests pass, 227 pass overall (2 pre-existing test_jobs failures,
lelab/ untouched), ruff clean at both py312 and py310 targets, and the B stage
still imports without Isaac present.

Co-Authored-By: Claude Opus 5 <noreply@anthropic.com>

File: lelab_sim/assets/omx_bimanual.urdf (robot description, URDF)
Before this commit: robot omx_bimanual, 19 links, 18 joints
Links:
- link left_link0: geometry collision mesh filename=../../frontend/public/omx-urdf/meshes/omx_f/follower_01_bas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 scale=0.001 0.001 0.001; visual mesh filename=../../frontend/public/omx-urdf/meshes/omx_f/follower_01_bas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 scale=0.001 0.001 0.001
- link left_link1: geometry collision mesh filename=../../frontend/public/omx-urdf/meshes/omx_f/follower_02_bas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 scale=0.001 0.001 0.001; visual mesh filename=../../frontend/public/omx-urdf/meshes/omx_f/follower_02_bas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 scale=0.001 0.001 0.001
- link left_link2: geometry collision mesh filename=../../frontend/public/omx-urdf/meshes/omx_f/follower_03_mid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 scale=0.001 0.001 0.001; visual mesh filename=../../frontend/public/omx-urdf/meshes/omx_f/follower_03_mid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 scale=0.001 0.001 0.001
- link left_link3: geometry collision mesh filename=../../frontend/public/omx-urdf/meshes/omx_f/follower_04_mid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 scale=0.001 0.001 0.001; visual mesh filename=../../frontend/public/omx-urdf/meshes/omx_f/follower_04_mid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 scale=0.001 0.001 0.001
- link left_link4: geometry collision mesh filename=../../frontend/public/omx-urdf/meshes/omx_f/follower_05_tip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 scale=0.001 0.001 0.001; visual mesh filename=../../frontend/public/omx-urdf/meshes/omx_f/follower_05_tip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 scale=0.001 0.001 0.001
- link left_link5: geometry collision mesh filename=../../frontend/public/omx-urdf/meshes/omx_f/follower_06_pan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 scale=0.001 0.001 0.001; visual mesh filename=../../frontend/public/omx-urdf/meshes/omx_f/follower_06_pan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 scale=0.001 0.001 0.001
- link left_link6: geometry collision mesh filename=../../frontend/public/omx-urdf/meshes/omx_f/follower_07_gri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 scale=0.001 0.001 0.001; visual mesh filename=../../frontend/public/omx-urdf/meshes/omx_f/follower_07_gri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 scale=0.001 0.001 0.001
- link left_link7: geometry collision mesh filename=../../frontend/public/omx-urdf/meshes/omx_f/follower_08_gri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 scale=0.001 0.001 0.001; visual mesh filename=../../frontend/public/omx-urdf/meshes/omx_f/follower_08_gri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 scale=0.001 0.001 0.001
- link right_link0: geometry collision mesh filename=../../frontend/public/omx-urdf/meshes/omx_f/follower_01_bas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 scale=0.001 0.001 0.001; visual mesh filename=../../frontend/public/omx-urdf/meshes/omx_f/follower_01_bas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 scale=0.001 0.001 0.001
- link right_link1: geometry collision mesh filename=../../frontend/public/omx-urdf/meshes/omx_f/follower_02_bas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 scale=0.001 0.001 0.001; visual mesh filename=../../frontend/public/omx-urdf/meshes/omx_f/follower_02_bas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 scale=0.001 0.001 0.001
- link right_link2: geometry collision mesh filename=../../frontend/public/omx-urdf/meshes/omx_f/follower_03_mid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 scale=0.001 0.001 0.001; visual mesh filename=../../frontend/public/omx-urdf/meshes/omx_f/follower_03_mid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 scale=0.001 0.001 0.001
- link right_link3: geometry collision mesh filename=../../frontend/public/omx-urdf/meshes/omx_f/follower_04_mid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 scale=0.001 0.001 0.001; visual mesh filename=../../frontend/public/omx-urdf/meshes/omx_f/follower_04_mid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 scale=0.001 0.001 0.001
- link right_link4: geometry collision mesh filename=../../frontend/public/omx-urdf/meshes/omx_f/follower_05_tip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 scale=0.001 0.001 0.001; visual mesh filename=../../frontend/public/omx-urdf/meshes/omx_f/follower_05_tip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 scale=0.001 0.001 0.001
- link right_link5: geometry collision mesh filename=../../frontend/public/omx-urdf/meshes/omx_f/follower_06_pan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 scale=0.001 0.001 0.001; visual mesh filename=../../frontend/public/omx-urdf/meshes/omx_f/follower_06_pan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 scale=0.001 0.001 0.001
- link right_link6: geometry collision mesh filename=../../frontend/public/omx-urdf/meshes/omx_f/follower_07_gri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 scale=0.001 0.001 0.001; visual mesh filename=../../frontend/public/omx-urdf/meshes/omx_f/follower_07_gri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 scale=0.001 0.001 0.001
- link right_link7: geometry collision mesh filename=../../frontend/public/omx-urdf/meshes/omx_f/follower_08_gri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 scale=0.001 0.001 0.001; visual mesh filename=../../frontend/public/omx-urdf/meshes/omx_f/follower_08_gri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 scale=0.001 0.001 0.001
Joints:
- joint left_gripper_joint_2: limit lower=-6.283185307179586 upper=6.283185307179586 effort=1000 velocity=4.8 -> lower=-1.7450 upper=-0.0000 effort=1000 velocity=4.8
- joint right_gripper_joint_2: limit lower=-6.283185307179586 upper=6.283185307179586 effort=1000 velocity=4.8 -> lower=-1.7450 upper=-0.0000 effort=1000 velocity=4.8
